Commit message: add: leo based structure

File: pixkit_description/urdf/vehicle.xacro (robot description, xacro)
@@ -1,3 +1,8 @@
-<?xml version="1.0"?>
+<?xml version="1.0" encoding="utf-8"?>
+<robot xmlns:xacro="http://www.ros.org/wiki/xacro"
+       name="pixkit">
+  <xacro:include filename="$(find pixkit_description)/urdf/macros.xacro"/>
+</robot>
+<!-- <?xml version="1.0"?>
 <robot xmlns:xacro="http://ros.org/wiki/xacro" name="pixkit_vehicle">
   <!-- load parameter -->
@@ -12,11 +17,3 @@
     </visual>
   </link>
-  <!-- <link name="base_link">
-    <visual>
-      <origin xyz="${vehicle_info['/**']['ros__parameters']['wheel_base']/2.0} 0 0" rpy="${pi/2.0} 0 ${pi}"/>
-      <geometry>
-        <mesh filename="package://pixkit_description/mesh/lexus.dae" scale="1 1 1"/>
-      </geometry>
-    </visual>
-  </link> -->
-</robot>
+</robot> -->
