Commit message: fix: forking xacro

File: pixkit_description/urdf/macros.xacro (robot description, xacro)
@@ -1,15 +1,13 @@
 <?xml version="1.0" encoding="utf-8"?>
 <robot xmlns:xacro="http://www.ros.org/wiki/xacro">
-  <xacro:macro name="vehicle_info" value="${xacro.load_yaml('$(find pixkit_description)/config/vehicle_info.param.yaml')}"/>
-    <xacro:macro name="base_link" params="name">
-        <link name="base_link">
-            <visual>
-            <origin xyz="-0.25 0.0 0.1" rpy="0 0 ${pi/2.0}"/>
-            <geometry>
-                <mesh filename="package://pixkit_description/mesh/hooke.dae" scale="0.001 0.001 0.001"/>
-            </geometry>
-            </visual>
-        </link>
-    </xacro:macro>
+    <xacro:macro name="pixkit" value="${xacro.load_yaml('$(find pixkit_description)/config/vehicle_info.param.yaml')}"/>
+    <link name="base_link">
+      <visual>
+        <origin xyz="-0.25 0.0 0.1" rpy="0 0 ${pi/2.0}"/>
+        <geometry>
+          <mesh filename="package://pixkit_description/mesh/hooke.dae" scale="0.001 0.001 0.001"/>
+        </geometry>
+      </visual>
+    </link>
   </xacro:macro>
 </robot>

Commit message: fix:scale

File: pixkit_description/urdf/macros.xacro (robot description, xacro)
@@ -1,12 +1,33 @@
 <?xml version="1.0" encoding="utf-8"?>
 <robot xmlns:xacro="http://www.ros.org/wiki/xacro">
-    <xacro:macro name="pixkit" value="${xacro.load_yaml('$(find pixkit_description)/config/vehicle_info.param.yaml')}"/>
-    <link name="base_link">
+  <xacro:macro name="pixkit"
+               params="default_antenna:=false
+                       rockers_fixed:=true
+                       footprint_link:=false
+                       link_prefix:=''
+                       joint_prefix:=''
+                       imu_translation:='0.0628 -0.0314 -0.0393'">
+    <!-- LINKS -->
+    <!-- Simple base_link with hooke visualization -->
+    <link name="${link_prefix}base_link">
+      <inertial>
+        <mass value="1.0"/>
+        <origin xyz="0 0 0"/>
+        <inertia
+          ixx="0.01" ixy="0" ixz="0"
+          iyy="0.01" iyz="0"
+          izz="0.01"/>
+      </inertial>
       <visual>
-        <origin xyz="-0.25 0.0 0.1" rpy="0 0 ${pi/2.0}"/>
+      <origin xyz="-0.25 0.0 0.1" rpy="0 0 ${pi/2.0}"/>
         <geometry>
-          <mesh filename="package://pixkit_description/mesh/hooke.dae" scale="0.001 0.001 0.001"/>
+          <mesh filename="package://pixkit_description/mesh/hooke.dae"/>
         </geometry>
       </visual>
+      <collision>
+        <geometry>
+          <box size="0.5 0.3 0.2"/>
+        </geometry>
+      </collision>
     </link>
   </xacro:macro>

Commit message: local path

File: pixkit_description/urdf/macros.xacro (robot description, xacro)
@@ -22,5 +22,5 @@
       <origin xyz="-0.25 0.0 0.1" rpy="0 0 ${pi/2.0}"/>
         <geometry>
-          <mesh filename="package://pixkit_description/mesh/hooke.dae"/>
+          <mesh filename="/home/stask/autoware_data/pixkit_launch/pixkit_description/mesh/hooke.dae"/>
         </geometry>
       </visual>

Commit message: absolute path

File: pixkit_description/urdf/macros.xacro (robot description, xacro)
@@ -22,5 +22,5 @@
       <origin xyz="-0.25 0.0 0.1" rpy="0 0 ${pi/2.0}"/>
         <geometry>
-          <mesh filename="/home/stask/autoware_data/pixkit_launch/pixkit_description/mesh/hooke.dae"/>
+          <mesh filename="package://pixkit_description/mesh/hooke.dae"/>
         </geometry>
       </visual>
